File: nerve_pcb_can.kicad_sch (KiCad schematic)
At the start: 6 parts, among them J7 CAN1, J8 CAN2, U5 TJA1051T/3, U6 TJA1051T/3

Commit message: Simplify clock circuits
Parts:
- renumbered R25 to R22, R26 to R23
Changed lines of the file:
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@@
 		(on_board yes)
 		(dnp no)
-		(property "Reference" "R25"
+		(property "Reference" "R22"
 			(at 138.684 110.49 0)
 			(effects
@@
 			(project "nerve_pcb"
 				(path "/c0277862-b3f2-4e0e-986f-34702f0543f0/4fcd2c12-d66e-4aef-b6ae-64082d99e104"
-					(reference "R25")
+					(reference "R22")
 					(unit 1)
 				)
@@
 		(on_board yes)
 		(dnp no)
-		(property "Reference" "R26"
+		(property "Reference" "R23"
 			(at 214.884 110.49 0)
 			(effects
@@
 			(project "nerve_pcb"
 				(path "/c0277862-b3f2-4e0e-986f-34702f0543f0/4fcd2c12-d66e-4aef-b6ae-64082d99e104"
-					(reference "R26")
-					(unit 1)
-				)
+					(reference "R23")
+					(unit 1)
+				)

Commit message: Update IMU clock circuit and cleanup
Parts:
- renumbered R22 to R20, R23 to R21
Changed lines of the file:
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@@
 		(on_board yes)
 		(dnp no)
-		(property "Reference" "R22"
+		(property "Reference" "R20"
 			(at 138.684 110.49 0)
 			(effects
@@
 			(project "nerve_pcb"
 				(path "/c0277862-b3f2-4e0e-986f-34702f0543f0/4fcd2c12-d66e-4aef-b6ae-64082d99e104"
-					(reference "R22")
+					(reference "R20")
 					(unit 1)
 				)
@@
 		(on_board yes)
 		(dnp no)
-		(property "Reference" "R23"
+		(property "Reference" "R21"
 			(at 214.884 110.49 0)
 			(effects
@@
 			(project "nerve_pcb"
 				(path "/c0277862-b3f2-4e0e-986f-34702f0543f0/4fcd2c12-d66e-4aef-b6ae-64082d99e104"
-					(reference "R23")
-					(unit 1)
-				)
+					(reference "R21")
+					(unit 1)
+				)

Commit message: Cleanup and update 2x10 Radio connector
Parts:
- renumbered J7 to J8, J8 to J9
Changed lines of the file:
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@@
 		(dnp no)
 		(fields_autoplaced yes)
-		(property "Reference" "#PWR083"
+		(property "Reference" "#PWR075"
 			(at 111.76 127 0)
 			(effects
@@
 			(project "nerve_pcb"
 				(path "/c0277862-b3f2-4e0e-986f-34702f0543f0/4fcd2c12-d66e-4aef-b6ae-64082d99e104"
-					(reference "#PWR083")
+					(reference "#PWR075")
 					(unit 1)
 				)
@@
 		(on_board yes)
 		(dnp no)
-		(property "Reference" "#PWR079"
+		(property "Reference" "#PWR071"
 			(at 86.36 101.6 0)
 			(effects
@@
 			(project "nerve_pcb"
 				(path "/c0277862-b3f2-4e0e-986f-34702f0543f0/4fcd2c12-d66e-4aef-b6ae-64082d99e104"
-					(reference "#PWR079")
+					(reference "#PWR071")
 					(unit 1)
 				)
@@
 		(on_board yes)
 		(dnp no)
-		(property "Reference" "#PWR080"
+		(property "Reference" "#PWR072"
 			(at 111.76 101.6 0)
 			(effects
@@
 			(project "nerve_pcb"
 				(path "/c0277862-b3f2-4e0e-986f-34702f0543f0/4fcd2c12-d66e-4aef-b6ae-64082d99e104"
-					(reference "#PWR080")
+					(reference "#PWR072")
 					(unit 1)
 				)
@@
 		(on_board yes)
 		(dnp no)
-		(property "Reference" "#PWR081"
+		(property "Reference" "#PWR073"
 			(at 162.56 101.6 0)
 			(effects
@@
 			(project "nerve_pcb"
 				(path "/c0277862-b3f2-4e0e-986f-34702f0543f0/4fcd2c12-d66e-4aef-b6ae-64082d99e104"
-					(reference "#PWR081")
+					(reference "#PWR073")
 					(unit 1)
 				)
@@
 		(on_board yes)
 		(dnp no)
-		(property "Reference" "#PWR082"
+		(property "Reference" "#PWR074"
 			(at 187.96 101.6 0)
 			(effects
@@
 			(project "nerve_pcb"
 				(path "/c0277862-b3f2-4e0e-986f-34702f0543f0/4fcd2c12-d66e-4aef-b6ae-64082d99e104"
-					(reference "#PWR082")
+					(reference "#PWR074")
 					(unit 1)
 				)
@@
 		(on_board yes)
 		(dnp no)
-		(property "Reference" "J7"
+		(property "Reference" "J8"
 			(at 153.416 106.68 0)
 			(effects
@@
 			(project "nerve_pcb"
 				(path "/c0277862-b3f2-4e0e-986f-34702f0543f0/4fcd2c12-d66e-4aef-b6ae-64082d99e104"
-					(reference "J7")
+					(reference "J8")
 					(unit 1)
 				)
@@
 		(on_board yes)
 		(dnp no)
-		(property "Reference" "J8"
+		(property "Reference" "J9"
 			(at 229.616 106.68 0)
 			(effects
@@
 			(project "nerve_pcb"
 				(path "/c0277862-b3f2-4e0e-986f-34702f0543f0/4fcd2c12-d66e-4aef-b6ae-64082d99e104"
-					(reference "J8")
+					(reference "J9")
 					(unit 1)
 				)
@@
 		(dnp no)
 		(fields_autoplaced yes)
-		(property "Reference" "#PWR084"
+		(property "Reference" "#PWR076"
 			(at 187.96 127 0)
 			(effects
@@
 			(project "nerve_pcb"
 				(path "/c0277862-b3f2-4e0e-986f-34702f0543f0/4fcd2c12-d66e-4aef-b6ae-64082d99e104"
-					(reference "#PWR084")
-					(unit 1)
-				)
+					(reference "#PWR076")
+					(unit 1)
+				)

Commit message: Add WS2812Bs
Parts:
- renumbered U5 to U6, U6 to U7
Changed lines of the file:
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@@
 		(dnp no)
 		(fields_autoplaced yes)
-		(property "Reference" "#PWR075"
+		(property "Reference" "#PWR082"
 			(at 111.76 127 0)
 			(effects
@@
 			(project "nerve_pcb"
 				(path "/c0277862-b3f2-4e0e-986f-34702f0543f0/4fcd2c12-d66e-4aef-b6ae-64082d99e104"
-					(reference "#PWR075")
+					(reference "#PWR082")
 					(unit 1)
 				)
@@
 		(on_board yes)
 		(dnp no)
-		(property "Reference" "#PWR071"
+		(property "Reference" "#PWR078"
 			(at 86.36 101.6 0)
 			(effects
@@
 			(project "nerve_pcb"
 				(path "/c0277862-b3f2-4e0e-986f-34702f0543f0/4fcd2c12-d66e-4aef-b6ae-64082d99e104"
-					(reference "#PWR071")
+					(reference "#PWR078")
 					(unit 1)
 				)
@@
 		(on_board yes)
 		(dnp no)
-		(property "Reference" "U6"
+		(property "Reference" "U7"
 			(at 198.882 98.298 0)
 			(effects
@@
 			(project "nerve_pcb"
 				(path "/c0277862-b3f2-4e0e-986f-34702f0543f0/4fcd2c12-d66e-4aef-b6ae-64082d99e104"
-					(reference "U6")
+					(reference "U7")
 					(unit 1)
 				)
@@
 		(on_board yes)
 		(dnp no)
-		(property "Reference" "#PWR072"
+		(property "Reference" "#PWR079"
 			(at 111.76 101.6 0)
 			(effects
@@
 			(project "nerve_pcb"
 				(path "/c0277862-b3f2-4e0e-986f-34702f0543f0/4fcd2c12-d66e-4aef-b6ae-64082d99e104"
-					(reference "#PWR072")
+					(reference "#PWR079")
 					(unit 1)
 				)
@@
 		(on_board yes)
 		(dnp no)
-		(property "Reference" "#PWR073"
+		(property "Reference" "#PWR080"
 			(at 162.56 101.6 0)
 			(effects
@@
 			(project "nerve_pcb"
 				(path "/c0277862-b3f2-4e0e-986f-34702f0543f0/4fcd2c12-d66e-4aef-b6ae-64082d99e104"
-					(reference "#PWR073")
+					(reference "#PWR080")
 					(unit 1)
 				)
@@
 		(on_board yes)
 		(dnp no)
-		(property "Reference" "#PWR074"
+		(property "Reference" "#PWR081"
 			(at 187.96 101.6 0)
 			(effects
@@
 			(project "nerve_pcb"
 				(path "/c0277862-b3f2-4e0e-986f-34702f0543f0/4fcd2c12-d66e-4aef-b6ae-64082d99e104"
-					(reference "#PWR074")
+					(reference "#PWR081")
 					(unit 1)
 				)
@@
 		(on_board yes)
 		(dnp no)
-		(property "Reference" "U5"
+		(property "Reference" "U6"
 			(at 122.682 98.298 0)
 			(effects
@@
 			(project ""
 				(path "/c0277862-b3f2-4e0e-986f-34702f0543f0/4fcd2c12-d66e-4aef-b6ae-64082d99e104"
-					(reference "U5")
+					(reference "U6")
 					(unit 1)
 				)
@@
 		(dnp no)
 		(fields_autoplaced yes)
-		(property "Reference" "#PWR076"
+		(property "Reference" "#PWR083"
 			(at 187.96 127 0)
 			(effects
@@
 			(project "nerve_pcb"
 				(path "/c0277862-b3f2-4e0e-986f-34702f0543f0/4fcd2c12-d66e-4aef-b6ae-64082d99e104"
-					(reference "#PWR076")
-					(unit 1)
-				)
+					(reference "#PWR083")
+					(unit 1)
+				)

Commit message: Fix BNO085 circuit for SPI
Parts:
- renumbered R20 to R19, R21 to R20
Changed lines of the file:
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@@
 		(dnp no)
 		(fields_autoplaced yes)
-		(property "Reference" "#PWR082"
+		(property "Reference" "#PWR081"
 			(at 111.76 127 0)
 			(effects
@@
 			(project "nerve_pcb"
 				(path "/c0277862-b3f2-4e0e-986f-34702f0543f0/4fcd2c12-d66e-4aef-b6ae-64082d99e104"
-					(reference "#PWR082")
+					(reference "#PWR081")
 					(unit 1)
 				)
@@
 		(on_board yes)
 		(dnp no)
-		(property "Reference" "#PWR078"
+		(property "Reference" "#PWR077"
 			(at 86.36 101.6 0)
 			(effects
@@
 			(project "nerve_pcb"
 				(path "/c0277862-b3f2-4e0e-986f-34702f0543f0/4fcd2c12-d66e-4aef-b6ae-64082d99e104"
-					(reference "#PWR078")
+					(reference "#PWR077")
 					(unit 1)
 				)
@@
 		(on_board yes)
 		(dnp no)
-		(property "Reference" "R20"
+		(property "Reference" "R19"
 			(at 138.684 110.49 0)
 			(effects
@@
 			(project "nerve_pcb"
 				(path "/c0277862-b3f2-4e0e-986f-34702f0543f0/4fcd2c12-d66e-4aef-b6ae-64082d99e104"
-					(reference "R20")
+					(reference "R19")
 					(unit 1)
 				)
@@
 		(on_board yes)
 		(dnp no)
-		(property "Reference" "#PWR079"
+		(property "Reference" "#PWR078"
 			(at 111.76 101.6 0)
 			(effects
@@
 			(project "nerve_pcb"
 				(path "/c0277862-b3f2-4e0e-986f-34702f0543f0/4fcd2c12-d66e-4aef-b6ae-64082d99e104"
-					(reference "#PWR079")
+					(reference "#PWR078")
 					(unit 1)
 				)
@@
 		(on_board yes)
 		(dnp no)
-		(property "Reference" "#PWR080"
+		(property "Reference" "#PWR079"
 			(at 162.56 101.6 0)
 			(effects
@@
 			(project "nerve_pcb"
 				(path "/c0277862-b3f2-4e0e-986f-34702f0543f0/4fcd2c12-d66e-4aef-b6ae-64082d99e104"
-					(reference "#PWR080")
+					(reference "#PWR079")
 					(unit 1)
 				)
@@
 		(on_board yes)
 		(dnp no)
-		(property "Reference" "#PWR081"
+		(property "Reference" "#PWR080"
 			(at 187.96 101.6 0)
 			(effects
@@
 			(project "nerve_pcb"
 				(path "/c0277862-b3f2-4e0e-986f-34702f0543f0/4fcd2c12-d66e-4aef-b6ae-64082d99e104"
-					(reference "#PWR081")
+					(reference "#PWR080")
 					(unit 1)
 				)
@@
 		(on_board yes)
 		(dnp no)
-		(property "Reference" "R21"
+		(property "Reference" "R20"
 			(at 214.884 110.49 0)
 			(effects
@@
 			(project "nerve_pcb"
 				(path "/c0277862-b3f2-4e0e-986f-34702f0543f0/4fcd2c12-d66e-4aef-b6ae-64082d99e104"
-					(reference "R21")
+					(reference "R20")
 					(unit 1)
 				)
@@
 		(dnp no)
 		(fields_autoplaced yes)
-		(property "Reference" "#PWR083"
+		(property "Reference" "#PWR082"
 			(at 187.96 127 0)
 			(effects
@@
 			(project "nerve_pcb"
 				(path "/c0277862-b3f2-4e0e-986f-34702f0543f0/4fcd2c12-d66e-4aef-b6ae-64082d99e104"
-					(reference "#PWR083")
-					(unit 1)
-				)
+					(reference "#PWR082")
+					(unit 1)
+				)
