File: nerve_pcb_baro.kicad_sch (KiCad schematic)
At the start: 7 parts, among them U5 BMP390

Commit message: Add minor decoupling caps
Parts:
- renumbered C22 to C25, C23 to C26
Changed lines of the file:
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@@
 		(dnp no)
 		(fields_autoplaced yes)
-		(property "Reference" "#PWR079"
+		(property "Reference" "#PWR082"
 			(at 137.16 115.57 0)
 			(effects
@@
 			(project "nerve_pcb"
 				(path "/c0277862-b3f2-4e0e-986f-34702f0543f0/9de129d2-0f7b-4a2d-85ad-214e335f6288"
-					(reference "#PWR079")
+					(reference "#PWR082")
 					(unit 1)
 				)
@@
 		(on_board yes)
 		(dnp no)
-		(property "Reference" "C22"
+		(property "Reference" "C25"
 			(at 148.59 68.58 0)
 			(effects
@@
 			(project "nerve_pcb"
 				(path "/c0277862-b3f2-4e0e-986f-34702f0543f0/9de129d2-0f7b-4a2d-85ad-214e335f6288"
-					(reference "C22")
+					(reference "C25")
 					(unit 1)
 				)
@@
 		(on_board yes)
 		(dnp no)
-		(property "Reference" "#PWR076"
+		(property "Reference" "#PWR079"
 			(at 184.15 92.71 0)
 			(effects
@@
 			(project "nerve_pcb"
 				(path "/c0277862-b3f2-4e0e-986f-34702f0543f0/9de129d2-0f7b-4a2d-85ad-214e335f6288"
-					(reference "#PWR076")
+					(reference "#PWR079")
 					(unit 1)
 				)
@@
 		(on_board yes)
 		(dnp no)
-		(property "Reference" "C23"
+		(property "Reference" "C26"
 			(at 161.29 68.58 0)
 			(effects
@@
 			(project "nerve_pcb"
 				(path "/c0277862-b3f2-4e0e-986f-34702f0543f0/9de129d2-0f7b-4a2d-85ad-214e335f6288"
-					(reference "C23")
+					(reference "C26")
 					(unit 1)
 				)
@@
 		(on_board yes)
 		(dnp no)
-		(property "Reference" "#PWR075"
+		(property "Reference" "#PWR078"
 			(at 156.21 92.71 0)
 			(effects
@@
 			(project "nerve_pcb"
 				(path "/c0277862-b3f2-4e0e-986f-34702f0543f0/9de129d2-0f7b-4a2d-85ad-214e335f6288"
-					(reference "#PWR075")
+					(reference "#PWR078")
 					(unit 1)
 				)
@@
 		(on_board yes)
 		(dnp no)
-		(property "Reference" "#PWR073"
+		(property "Reference" "#PWR076"
 			(at 158.75 67.31 0)
 			(effects
@@
 			(project "nerve_pcb"
 				(path "/c0277862-b3f2-4e0e-986f-34702f0543f0/9de129d2-0f7b-4a2d-85ad-214e335f6288"
-					(reference "#PWR073")
+					(reference "#PWR076")
 					(unit 1)
 				)
@@
 		(dnp no)
 		(fields_autoplaced yes)
-		(property "Reference" "#PWR074"
+		(property "Reference" "#PWR077"
 			(at 158.75 82.55 0)
 			(effects
@@
 			(project "nerve_pcb"
 				(path "/c0277862-b3f2-4e0e-986f-34702f0543f0/9de129d2-0f7b-4a2d-85ad-214e335f6288"
-					(reference "#PWR074")
+					(reference "#PWR077")
 					(unit 1)
 				)
@@
 		(on_board yes)
 		(dnp no)
-		(property "Reference" "#PWR077"
+		(property "Reference" "#PWR080"
 			(at 123.19 96.52 0)
 			(effects
@@
 			(project "nerve_pcb"
 				(path "/c0277862-b3f2-4e0e-986f-34702f0543f0/9de129d2-0f7b-4a2d-85ad-214e335f6288"
-					(reference "#PWR077")
+					(reference "#PWR080")
 					(unit 1)
 				)
@@
 		(on_board yes)
 		(dnp no)
-		(property "Reference" "#PWR078"
+		(property "Reference" "#PWR081"
 			(at 114.3 100.33 0)
 			(effects
@@
 			(project "nerve_pcb"
 				(path "/c0277862-b3f2-4e0e-986f-34702f0543f0/9de129d2-0f7b-4a2d-85ad-214e335f6288"
-					(reference "#PWR078")
+					(reference "#PWR081")
 					(unit 1)
 				)
@@
 		(dnp no)
 		(fields_autoplaced yes)
-		(property "Reference" "#PWR080"
+		(property "Reference" "#PWR083"
 			(at 171.45 118.11 0)
 			(effects
@@
 			(project "nerve_pcb"
 				(path "/c0277862-b3f2-4e0e-986f-34702f0543f0/9de129d2-0f7b-4a2d-85ad-214e335f6288"
-					(reference "#PWR080")
-					(unit 1)
-				)
+					(reference "#PWR083")
+					(unit 1)
+				)

Commit message: Add WS2812B decoupling caps and PCB cleanup
Parts:
- renumbered C25 to C27, C26 to C28
Changed lines of the file:
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@@
 		(dnp no)
 		(fields_autoplaced yes)
-		(property "Reference" "#PWR082"
+		(property "Reference" "#PWR084"
 			(at 137.16 115.57 0)
 			(effects
@@
 			(project "nerve_pcb"
 				(path "/c0277862-b3f2-4e0e-986f-34702f0543f0/9de129d2-0f7b-4a2d-85ad-214e335f6288"
-					(reference "#PWR082")
+					(reference "#PWR084")
 					(unit 1)
 				)
@@
 		(on_board yes)
 		(dnp no)
-		(property "Reference" "C25"
+		(property "Reference" "C27"
 			(at 148.59 68.58 0)
 			(effects
@@
 			(project "nerve_pcb"
 				(path "/c0277862-b3f2-4e0e-986f-34702f0543f0/9de129d2-0f7b-4a2d-85ad-214e335f6288"
-					(reference "C25")
+					(reference "C27")
 					(unit 1)
 				)
@@
 		(on_board yes)
 		(dnp no)
-		(property "Reference" "#PWR079"
+		(property "Reference" "#PWR081"
 			(at 184.15 92.71 0)
 			(effects
@@
 			(project "nerve_pcb"
 				(path "/c0277862-b3f2-4e0e-986f-34702f0543f0/9de129d2-0f7b-4a2d-85ad-214e335f6288"
-					(reference "#PWR079")
+					(reference "#PWR081")
 					(unit 1)
 				)
@@
 		(on_board yes)
 		(dnp no)
-		(property "Reference" "C26"
+		(property "Reference" "C28"
 			(at 161.29 68.58 0)
 			(effects
@@
 			(project "nerve_pcb"
 				(path "/c0277862-b3f2-4e0e-986f-34702f0543f0/9de129d2-0f7b-4a2d-85ad-214e335f6288"
-					(reference "C26")
+					(reference "C28")
 					(unit 1)
 				)
@@
 		(on_board yes)
 		(dnp no)
-		(property "Reference" "#PWR078"
+		(property "Reference" "#PWR080"
 			(at 156.21 92.71 0)
 			(effects
@@
 			(project "nerve_pcb"
 				(path "/c0277862-b3f2-4e0e-986f-34702f0543f0/9de129d2-0f7b-4a2d-85ad-214e335f6288"
-					(reference "#PWR078")
+					(reference "#PWR080")
 					(unit 1)
 				)
@@
 		(on_board yes)
 		(dnp no)
-		(property "Reference" "#PWR076"
+		(property "Reference" "#PWR078"
 			(at 158.75 67.31 0)
 			(effects
@@
 			(project "nerve_pcb"
 				(path "/c0277862-b3f2-4e0e-986f-34702f0543f0/9de129d2-0f7b-4a2d-85ad-214e335f6288"
-					(reference "#PWR076")
+					(reference "#PWR078")
 					(unit 1)
 				)
@@
 		(dnp no)
 		(fields_autoplaced yes)
-		(property "Reference" "#PWR077"
+		(property "Reference" "#PWR079"
 			(at 158.75 82.55 0)
 			(effects
@@
 			(project "nerve_pcb"
 				(path "/c0277862-b3f2-4e0e-986f-34702f0543f0/9de129d2-0f7b-4a2d-85ad-214e335f6288"
-					(reference "#PWR077")
+					(reference "#PWR079")
 					(unit 1)
 				)
@@
 		(on_board yes)
 		(dnp no)
-		(property "Reference" "#PWR080"
+		(property "Reference" "#PWR082"
 			(at 123.19 96.52 0)
 			(effects
@@
 			(project "nerve_pcb"
 				(path "/c0277862-b3f2-4e0e-986f-34702f0543f0/9de129d2-0f7b-4a2d-85ad-214e335f6288"
-					(reference "#PWR080")
+					(reference "#PWR082")
 					(unit 1)
 				)
@@
 		(on_board yes)
 		(dnp no)
-		(property "Reference" "#PWR081"
+		(property "Reference" "#PWR083"
 			(at 114.3 100.33 0)
 			(effects
@@
 			(project "nerve_pcb"
 				(path "/c0277862-b3f2-4e0e-986f-34702f0543f0/9de129d2-0f7b-4a2d-85ad-214e335f6288"
-					(reference "#PWR081")
+					(reference "#PWR083")
 					(unit 1)
 				)
@@
 		(dnp no)
 		(fields_autoplaced yes)
-		(property "Reference" "#PWR083"
+		(property "Reference" "#PWR085"
 			(at 171.45 118.11 0)
 			(effects
@@
 			(project "nerve_pcb"
 				(path "/c0277862-b3f2-4e0e-986f-34702f0543f0/9de129d2-0f7b-4a2d-85ad-214e335f6288"
-					(reference "#PWR083")
-					(unit 1)
-				)
+					(reference "#PWR085")
+					(unit 1)
+				)
